File: PCB/Rhenium-Hub.kicad_pcb (KiCad board)
At the start: 2 copper layers, 48 x 57 mm, 27 parts, among them J1 USB_A, J2 USB_A, J3 USB_C_Receptacle_USB2.0_16P, J4 USB_C_Receptacle_USB2.0_16P, J5 USB_C_Receptacle_USB2.0_16P, U1 USB2514B_Bi

Commit message: Updated the pcb
Parts:
- added C5: 0.1µF, Capacitor_SMD:C_0603_1608Metric, F.Cu at (120.7, 78.0)
- J1, J2: footprint Connector_USB:USB_A_CNCTech_1001-011-01101_Horizontal -> Connector_USB:USB_A_Molex_105057_Vertical
- moved J2 4.69 mm to (91.3, 83.5), turned to 90 degrees
- moved J1 4.62 mm to (90.6, 65.1), turned to 0 degrees
- moved G*** 4.20 mm to (107.2, 112.7) (x2)
- moved G*** 3.80 mm to (100.8, 83.3)
- moved G*** 0.98 mm to (118.3, 102.4)
- moved G*** 0.91 mm to (127.8, 105.6)
Routing:
- net GND: track 230.8 -> 249.8 mm, vias 4 -> 5
- net D2_N: track 8.16 -> 22.2 mm
- net D2_P: track 8.16 -> 21.6 mm
- net +5V: track 159.8 -> 150.1 mm
- net D1_P: track 21.0 -> 25.9 mm
- net D1_N: track 21.0 -> 24.5 mm
- net +3.3V: track 32.1 -> 31.1 mm
Other:
- board text added: "${REFERENCE}"

Commit message: hihi
Parts:
- removed the G*** at (127.8, 105.6)
Connections:
- U1 pad 10: +3.3V -> +3V3
- U1 pad 15: +3.3V -> +3V3
- U1 pad 23: +3.3V -> +3V3
- U1 pad 29: +3.3V -> +3V3
- U1 pad 36: +3.3V -> +3V3
- U1 pad 5: +3.3V -> +3V3
