File: PCB/Erbium.kicad_pcb (KiCad board)
At the start: 2 copper layers, 48 x 57 mm, 27 parts, among them J1 USB_A, J2 USB_A, J3 USB_C_Receptacle_USB2.0_16P, J4 USB_C_Receptacle_USB2.0_16P, J5 USB_C_Receptacle_USB2.0_16P, U1 USB2514B_Bi

Commit message: updated
Parts:
- removed C1, C2, C3, C4, C6: 0.1µF, Capacitor_SMD:C_0603_1608Metric
- added C10: 0.1µF, Capacitor_SMD:C_0603_1608Metric, F.Cu at (114.2, 87.2)
- added C11: 0.1µF, Capacitor_SMD:C_0603_1608Metric, F.Cu at (117.5, 87.2)
- added C12: 0.1µF, Capacitor_SMD:C_0603_1608Metric, F.Cu at (115.8, 87.2)
- added C9: 0.1µF, Capacitor_SMD:C_0603_1608Metric, F.Cu at (119.1, 87.2)
- added G***: LOGO, LOGO, F.Cu at (127.8, 100.8)
- R1, R2, R3, R4: value 5.1k -> 56k
- moved R2 2.40 mm to (93.6, 105.9)
- moved G*** 2.38 mm to (115.9, 102.4)
- moved R1 1.77 mm to (94.8, 92.2), turned to -90 degrees
- moved R4 0.78 mm to (93.7, 110.9)
- moved R3 0.45 mm to (93.8, 98.4)
Connections:
- C5 pad 2: +3.3V -> +3V3
- R1 pad 1: GND -> +5V
- R2 pad 1: GND -> +5V
- R3 pad 1: GND -> +5V
- R4 pad 1: GND -> +5V
- R5 pad 1: +3.3V -> +3V3
Routing:
- net +3V3: track 0.00 -> 41.1 mm, vias 0 -> 2
- net +3.3V: track 31.1 -> 0.00 mm
- net GND: track 249.8 -> 279.6 mm
- net +5V: track 150.1 -> 163.4 mm
- net Net-(J4-CC1): track 4.48 -> 2.48 mm
- net Net-(J3-CC1): track 2.36 -> 4.17 mm
- net Net-(J4-CC2): track 3.25 -> 2.41 mm
