File: PCB/Erbium.kicad_sch (KiCad schematic)
At the start: 22 parts, among them J1 USB_A, J2 USB_A, J3 USB_C_Receptacle_USB2.0_16P, J4 USB_C_Receptacle_USB2.0_16P, J5 USB_C_Receptacle_USB2.0_16P, U1 USB2514B_Bi

Commit message: updated
Parts:
- added J6: USB_A, symbol Connector:USB_A
- R1, R2, R3, R4: value 5.1k -> 56k
Connections:
- net +3.3V is gone; now on net +3V3: R5.1
- net +5V: now also R1.1, R2.1, R3.1, R4.1
- net GND: no longer R1.1, R2.1, R3.1, R4.1
Other:
- moved on the sheet: J1, J2
